Commit message: edited joints calibrator, added some folder for move_base's parameters to backup my work

File: oped_description/urdf/gazebo/accessories.urdf.xacro (robot description, xacro)
@@ -12,7 +12,7 @@
         <origin xyz="0.0 0.0 ${base_z_length / 2 + 0.04}" rpy="0 0 0"/>
     </xacro:hokuyo_utm30lx> -->
-    <!-- <gazebo reference="hokuyo_frame">
+    <gazebo reference="hokuyo_frame">
 		<material>Gazebo/FlatBlack</material>
-	</gazebo> -->
+	</gazebo>
     <gazebo reference="lidar_frame">
       <material>Gazebo/FlatBlack</material>

File: oped_description/urdf/oped.urdf (robot description, URDF)
Before this commit: robot oped, 24 links, 23 joints
Links:
- link base_inertia: mass 0.4 -> 0.7

File: oped_description/urdf/properties.urdf.xacro (robot description, xacro)
@@ -23,5 +23,5 @@
     <xacro:property name="lower_leg_z_length" value="0.0503" />
     <xacro:property name="base_mesh_path" value="package://oped_description/meshes/base.dae" />
-    <xacro:property name="base_mass" value="0.4" /> <!--0.65 tanpa kepala-->
+    <xacro:property name="base_mass" value="0.7" /> <!--0.65 tanpa kepala-->
     <xacro:property name="base_x_length" value="0.108" />
     <xacro:property name="base_y_length" value="0.058" />
