Commit message: change the urdf to x orientation

File: oped_description/urdf/accessories.urdf.xacro (robot description, xacro)
@@ -64,15 +64,15 @@
         <parent link="base_link"/>
         <child link="lidar_frame"/>
-        <origin xyz="0 0 0.077" rpy="0 0 0"/>
+        <origin xyz="-0.007 0 0.077" rpy="0 0 0"/>
     </joint>
     <link name="lidar_frame">
         <visual>
-            <origin xyz="0 0 -0.077" rpy="0 0 0"/>
+            <origin xyz="0.007 0 -0.067" rpy="0 0 0"/>
             <geometry>
-              <mesh filename="package://oped_description/meshes/ydlidar_x4.dae"/>
+              <mesh filename="package://oped_description/meshes/rplidar.dae"/>
             </geometry>
         </visual>
         <collision>
-            <origin xyz="-0.007 0 0" rpy="0 0 0"/>
+            <origin xyz="0 0 0.01" rpy="0 0 0"/>
             <geometry>
                 <cylinder length="0.0315" radius="0.035"/>

File: oped_description/urdf/gazebo/champ.urdf (robot description, URDF)
Before this commit: robot champ, 24 links, 23 joints
Links:
- link base_link: geometry collision mesh filename=package://oped_description/meshes/gazebo/base.stl scale=1.0 2.05555 1.0; visual mesh filename=package://oped_description/meshes/gazebo/base.stl scale=1.0 2.05555 1.0
Joints:
- joint lf_debug_joint: origin xyz=0.09213295 0.03910347 0 rpy=0 0 0 -> xyz=0.09213295 0.080379285 0 rpy=0 0 0
- joint lf_hip_joint: origin xyz=0.09213295 0.03910347 0 rpy=0 0 0 -> xyz=0.09213295 0.080379285 0 rpy=0 0 0
- joint lh_debug_joint: origin xyz=-0.09213295 0.03910347 0 rpy=0 0 0 -> xyz=-0.09213295 0.080379285 0 rpy=0 0 0
- joint lh_hip_joint: origin xyz=-0.09213295 0.03910347 0 rpy=0 0 0 -> xyz=-0.09213295 0.080379285 0 rpy=0 0 0
- joint rf_debug_joint: origin xyz=0.09213295 -0.03910347 0 rpy=0 0 0 -> xyz=0.09213295 -0.080379285 0 rpy=0 0 0
- joint rf_hip_joint: origin xyz=0.09213295 -0.03910347 0 rpy=0 0 0 -> xyz=0.09213295 -0.080379285 0 rpy=0 0 0
- joint rh_debug_joint: origin xyz=-0.09213295 -0.03910347 0 rpy=0 0 0 -> xyz=-0.09213295 -0.080379285 0 rpy=0 0 0
- joint rh_hip_joint: origin xyz=-0.09213295 -0.03910347 0 rpy=0 0 0 -> xyz=-0.09213295 -0.080379285 0 rpy=0 0 0

File: oped_description/urdf/gazebo/champ.urdf.xacro (robot description, xacro)
@@ -7,5 +7,5 @@
             <origin xyz="0 0 0" rpy="0 0 0" />
             <geometry>
-                <mesh filename="${base_mesh_path}" />
+                <mesh filename="${base_mesh_path}" scale="1.0 2.05555 1.0"/>
             </geometry>
         </collision>
@@ -13,5 +13,5 @@
             <origin xyz="0 0 0" rpy="0 0 0" />
             <geometry>
-                <mesh filename="package://oped_description/meshes/gazebo/base.stl" />
+                <mesh filename="${base_mesh_path}" scale="1.0 2.05555 1.0"/> <!--1.0 1.0 1.0-->
             </geometry>
             <material name="black" />

File: oped_description/urdf/gazebo/leg.urdf.xacro (robot description, xacro)
@@ -5,16 +5,20 @@
             <xacro:property name="base_to_hip_xyz" value="${base_to_hip_x} ${base_to_hip_y} 0" />
             <xacro:property name="hip_to_upper_leg" value="${hip_to_upper_leg_distance}" />
+            <xacro:property name="rotate_lower" value="0" />
         </xacro:if>
         <xacro:if value="${leg == 'lh'}">
             <xacro:property name="base_to_hip_xyz" value="-${base_to_hip_x} ${base_to_hip_y} 0" />
             <xacro:property name="hip_to_upper_leg" value="${hip_to_upper_leg_distance}" />
+            <xacro:property name="rotate_lower" value="-3.14159" />
         </xacro:if>
         <xacro:if value="${leg == 'rf'}">
             <xacro:property name="base_to_hip_xyz" value="${base_to_hip_x} -${base_to_hip_y} 0" />
             <xacro:property name="hip_to_upper_leg" value="-${hip_to_upper_leg_distance}" />
+            <xacro:property name="rotate_lower" value="0" />
         </xacro:if>
         <xacro:if value="${leg == 'rh'}">
             <xacro:property name="base_to_hip_xyz" value="-${base_to_hip_x} -${base_to_hip_y} 0" />
             <xacro:property name="hip_to_upper_leg" value="-${hip_to_upper_leg_distance}" />
+            <xacro:property name="rotate_lower" value="-3.14159" />
         </xacro:if>
         <link name="${leg}_hip_debug_link"/>
@@ -77,5 +81,5 @@
             </inertial>
             <collision>
-                <origin xyz="0 0 0" rpy="0 0 0" />
+                <origin xyz="0 0 0" rpy="0 0 ${rotate_lower}" />
                 <geometry>
                     <mesh filename="${lower_leg_mesh_path}" />
@@ -83,5 +87,5 @@
             </collision>
             <visual>
-                <origin xyz="0 0 0" rpy="0 0 0" />
+                <origin xyz="0 0 0" rpy="0 0 ${rotate_lower}" />
                 <geometry>
                     <mesh filename="${lower_leg_mesh_path}" />

File: oped_description/urdf/gazebo/properties.urdf.xacro (robot description, xacro)
@@ -2,5 +2,5 @@
 <robot xmlns:xacro="http://ros.org/wiki/xacro">
     <xacro:property name="base_to_hip_x" value="${0.175 * 0.526474}" />
-    <xacro:property name="base_to_hip_y" value="${0.105 * 0.372414}" />
+    <xacro:property name="base_to_hip_y" value="${0.105 * 0.765517}" />
     <xacro:property name="hip_to_upper_leg_distance" value="${0.06 * 0.507431}" />
     <xacro:property name="upper_leg_to_lower_leg_distance" value="${0.141 * 0.507431}" />
@@ -9,20 +9,20 @@
     <xacro:property name="hip_mass" value="${0.250 * 0.2}" /> <!--ubah-->
     <xacro:property name="hip_x_length" value="${0.112 * 0.526474}" />
-    <xacro:property name="hip_y_length" value="${0.08 * 0.372414}" />
+    <xacro:property name="hip_y_length" value="${0.08 * 0.765517}" />
     <xacro:property name="hip_z_length" value="${0.130 * 0.507431}" />
     <xacro:property name="upper_leg_mesh_path" value="package://oped_description/meshes/gazebo/upper_leg.stl" />
     <xacro:property name="upper_leg_mass" value="${0.125 * 0.2}" /> <!--ubah-->
     <xacro:property name="upper_leg_x_length" value="${0.5 * 0.526474}" />
-    <xacro:property name="upper_leg_y_length" value="${0.03 * 0.372414}" />
+    <xacro:property name="upper_leg_y_length" value="${0.03 * 0.765517}" /> <!--0.372414-->
     <xacro:property name="upper_leg_z_length" value="${0.1905 * 0.507431}" />
     <xacro:property name="lower_leg_mesh_path" value="package://oped_description/meshes/gazebo/lower_leg.stl" />
     <xacro:property name="lower_leg_mass" value="${0.125 * 0.2}" />
     <xacro:property name="lower_leg_x_length" value="${0.039 * 0.526474}" />
-    <xacro:property name="lower_leg_y_length" value="${0.022 * 0.372414}" />
+    <xacro:property name="lower_leg_y_length" value="${0.022 * 0.765517}" />
     <xacro:property name="lower_leg_z_length" value="${0.156 * 0.507431}" />
     <xacro:property name="base_mesh_path" value="package://oped_description/meshes/gazebo/base.stl" />
     <xacro:property name="base_mass" value="${2.0 * 0.2}" />
     <xacro:property name="base_x_length" value="${0.5 * 0.526474}" />
-    <xacro:property name="base_y_length" value="${0.29 * 0.372414}" />
+    <xacro:property name="base_y_length" value="${0.29 * 0.765517}" />
     <xacro:property name="base_z_length" value="${0.130 * 0.507431}" />
 </robot>

File: oped_description/urdf/leg.urdf.xacro (robot description, xacro)
@@ -6,4 +6,6 @@
             <xacro:property name="hip_to_upper_leg" value="${hip_to_upper_leg_distance}" />
             <xacro:property name="rotate_hip" value="-3.14159" />
+            <xacro:property name="rotate_upper" value="0" />
+            <xacro:property name="rotate_lower" value="0" />
         </xacro:if>
         <xacro:if value="${leg == 'lh'}">
@@ -11,4 +13,6 @@
             <xacro:property name="hip_to_upper_leg" value="${hip_to_upper_leg_distance}" />
             <xacro:property name="rotate_hip" value="-3.14159" />
+            <xacro:property name="rotate_upper" value="-3.14159" />
+            <xacro:property name="rotate_lower" value="-3.14159" />
         </xacro:if>
         <xacro:if value="${leg == 'rf'}">
@@ -16,4 +20,6 @@
             <xacro:property name="hip_to_upper_leg" value="-${hip_to_upper_leg_distance}" />
             <xacro:property name="rotate_hip" value="0" />
+            <xacro:property name="rotate_upper" value="0" />
+            <xacro:property name="rotate_lower" value="0" />
         </xacro:if>
         <xacro:if value="${leg == 'rh'}">
@@ -21,4 +27,6 @@
             <xacro:property name="hip_to_upper_leg" value="-${hip_to_upper_leg_distance}" />
             <xacro:property name="rotate_hip" value="0" />
+            <xacro:property name="rotate_upper" value="-3.14159" />
+            <xacro:property name="rotate_lower" value="-3.14159" />
         </xacro:if>
         <link name="${leg}_hip_debug_link"/>
@@ -56,5 +64,5 @@
             </inertial>
             <collision>
-                <origin xyz="0 0 0" rpy="0 0 0" />
+                <origin xyz="0 0 0" rpy="0 0 ${rotate_upper}" />
                 <geometry>
                     <xacro:if value="${leg == 'lf'}">
@@ -73,5 +81,5 @@
             </collision>
             <visual>
-                <origin xyz="0 0 0" rpy="0 0 0" />
+                <origin xyz="0 0 0" rpy="0 0 ${rotate_upper}" />
                 <geometry>
                     <xacro:if value="${leg == 'lf'}">
@@ -103,5 +111,5 @@
             </inertial>
             <collision>
-                <origin xyz="0 0 0" rpy="0 0 0" />
+                <origin xyz="0 0 0" rpy="0 0 ${rotate_lower}" />
                 <geometry>
                     <mesh filename="${lower_leg_mesh_path}"/>
@@ -109,5 +117,5 @@
             </collision>
             <visual>
-                <origin xyz="0 0 0" rpy="0 0 0" />
+                <origin xyz="0 0 0" rpy="0 0 ${rotate_lower}" />
                 <geometry>
                     <mesh filename="${lower_leg_mesh_path}"/>

File: oped_description/urdf/oped.urdf (robot description, URDF)
Before this commit: robot oped, 24 links, 23 joints
Links:
- link base_link: geometry collision mesh filename=package://oped_description/meshes/base_x.dae; visual mesh filename=package://oped_description/meshes/base_x.dae
- link lidar_frame: geometry collision cylinder length=0.0315 radius=0.035; visual mesh filename=package://oped_description/meshes/rplidar.dae
Joints:
- joint lf_debug_joint: origin xyz=0.074 0.04177 0 rpy=0 0 0 -> xyz=0.099 0.04177 0 rpy=0 0 0
- joint lf_hip_joint: origin xyz=0.074 0.04177 0 rpy=0 0 0 -> xyz=0.099 0.04177 0 rpy=0 0 0
- joint lh_debug_joint: origin xyz=-0.07 0.04177 0 rpy=0 0 0 -> xyz=-0.095 0.04177 0 rpy=0 0 0
- joint lh_hip_joint: origin xyz=-0.07 0.04177 0 rpy=0 0 0 -> xyz=-0.095 0.04177 0 rpy=0 0 0
- joint rf_debug_joint: origin xyz=0.074 -0.04177 0 rpy=0 0 0 -> xyz=0.099 -0.04177 0 rpy=0 0 0
- joint rf_hip_joint: origin xyz=0.074 -0.04177 0 rpy=0 0 0 -> xyz=0.099 -0.04177 0 rpy=0 0 0
- joint rh_debug_joint: origin xyz=-0.07 -0.04177 0 rpy=0 0 0 -> xyz=-0.095 -0.04177 0 rpy=0 0 0
- joint rh_hip_joint: origin xyz=-0.07 -0.04177 0 rpy=0 0 0 -> xyz=-0.095 -0.04177 0 rpy=0 0 0
- joint scan_joint: origin xyz=0 0 0.077 rpy=0 0 0 -> xyz=-0.007 0 0.077 rpy=0 0 0

File: oped_description/urdf/oped.urdf.xacro (robot description, xacro)
@@ -13,5 +13,5 @@
             <origin xyz="0 0 0" rpy="0 0 0" />
             <geometry>
-                <mesh filename="package://oped_description/meshes/base.dae"/>
+                <mesh filename="${base_mesh_path}"/>
             </geometry>
             <material name="black" />

File: oped_description/urdf/properties.urdf.xacro (robot description, xacro)
@@ -1,5 +1,5 @@
 <?xml version="1.0"?>
 <robot xmlns:xacro="http://ros.org/wiki/xacro">
-    <xacro:property name="base_to_hip_x" value="0.074" /> <!--0.072518-->
+    <xacro:property name="base_to_hip_x" value="0.099" /> <!--0.072518-->
     <xacro:property name="base_to_hip_y" value="0.04177" />
     <xacro:property name="hip_to_upper_leg_distance" value="0.052" />
@@ -22,5 +22,5 @@
     <xacro:property name="lower_leg_y_length" value="0.01351353" />
     <xacro:property name="lower_leg_z_length" value="0.0503" />
-    <xacro:property name="base_mesh_path" value="package://oped_description/meshes/base.dae" />
+    <xacro:property name="base_mesh_path" value="package://oped_description/meshes/base_x.dae" />
     <xacro:property name="base_mass" value="0.7" /> <!--0.65 tanpa kepala-->
     <xacro:property name="base_x_length" value="0.108" />
